File: kicad/Super Sixteen v1.sch (KiCad schematic (older format))
At the start: 110 parts, among them J1 Power Header, J2 Reset, J3 Clock In, J4 Gate Out, J5 Pitch Out, J6 Clock Out, J7 CV Out, Q1 2N3904, Q2 2N3904, Q3 2N3904, SW1 Load, SW10 S5, SW11 S6, SW12 S7, SW13 S2, SW14 S6, SW15 SW_Push, SW16 SW_Push, SW17 S3, SW18 S7, SW19 SW_Push, SW2 Repeat, SW20 SW_Push, SW21 S4, SW22 S8, SW23 SW_Push, SW24 SW_Push, SW3 Save, SW4 Mutate, SW5 Shift, SW6 GlideBtn, SW7 Play, SW8 Encoder, SW9 S1, U1 L7805, U2 W25Q80DVSN, U3 MCP4822, U4 TL072, U5 ATMEGA328P-PU, U6 MCP23S17, U7 MCP23S17, Y1 Crystal

Commit message: Updating schematic
Parts:
- C1: footprint (none) -> Capacitors_THT:CP_Radial_D4.0mm_P2.00mm
- C10, C9: footprint (none) -> Capacitors_THT:C_Disc_D3.0mm_W2.0mm_P2.50mm
- C3, C4: footprint (none) -> Capacitors_THT:CP_Radial_D5.0mm_P2.00mm
- D1, D2: footprint (none) -> Diodes_THT:D_5KPW_P7.62mm_Vertical_AnodeUp
- D10, D11, D12, D14, D15, D16, D17, D18, D19, D20, D21, D4, D5, D6, D7, D8, D9: footprint (none) -> LEDs:LED_D5.0mm
- J1: footprint (none) -> Socket_Strips:Socket_Strip_Straight_2x05_Pitch2.54mm
- J2: footprint (none) -> Socket_Strips:Socket_Strip_Angled_1x17_Pitch2.00mm
- L1, L2, L3: footprint (none) -> Inductors_THT:L_Axial_L6.6mm_D2.7mm_P10.16mm_Horizontal_Vishay_IM-2
- R1, R10, R11, R12, R13, R14, R15, R16, R17, R18, R19, R2, R20, R21, R22, R23, R24, R25, R26, R27, R3, R4, R5, R6, R7, R8, R9: footprint (none) -> Resistors_THT:R_Axial_DIN0207_L6.3mm_D2.5mm_P7.62mm_Horizontal
- RV1, RV2, RV3, RV4: footprint (none) -> Potentiometers:Potentiometer_Alps_RK09K_Horizontal
- SW1, SW10, SW11, SW12, SW13, SW14, SW15, SW16, SW17, SW18, SW19, SW20, SW21, SW22, SW23, SW24, SW3, SW5, SW6, SW7, SW8, SW9: footprint (none) -> Buttons_Switches_THT:SW_TH_Tactile_Omron_B3F-10xx
- SW2, SW4: footprint (none) -> Buttons_Switches_THT:SW_PUSH-12mm
- U1: footprint (none) -> TO_SOT_Packages_THT:TO-220-3_Horizontal
- U2: footprint (none) -> Housings_SOIC:SOIC-8_3.9x4.9mm_Pitch1.27mm
- U3, U4: footprint (none) -> Housings_DIP:DIP-8_W7.62mm_LongPads
- U6, U7: footprint (none) -> Housings_DIP:DIP-28_W15.24mm_LongPads
- Y1: footprint (none) -> Crystals:Crystal_HC49-4H_Vertical

Commit message: Updating schematic and PCB
Parts:
- removed C3, C4: 25uF, Capacitors_THT:CP_Radial_D5.0mm_P2.00mm, symbol CP1_Small
- removed D1, D2: D, Diodes_THT:D_5KPW_P7.62mm_Vertical_AnodeUp, symbol D
- removed D13: BA56-12YWA, symbol BA56-12YWA-RESCUE-Super_Sixteen_v1
- removed D22, D23: D, symbol D
- removed J1: Power Header, Socket_Strips:Socket_Strip_Straight_2x05_Pitch2.54mm, symbol Conn_02x05_Row_Letter_Last
- removed L1, L2: L, Inductors_THT:L_Axial_L6.6mm_D2.7mm_P10.16mm_Horizontal_Vishay_IM-2, symbol L
- removed R23, R25: R, Resistors_THT:R_Axial_DIN0207_L6.3mm_D2.5mm_P7.62mm_Horizontal, symbol R
- removed SW1: Load, Buttons_Switches_THT:SW_TH_Tactile_Omron_B3F-10xx, symbol SW_Push
- removed SW10: S5, Buttons_Switches_THT:SW_TH_Tactile_Omron_B3F-10xx, symbol SW_Push
- removed SW11, SW14: S6, Buttons_Switches_THT:SW_TH_Tactile_Omron_B3F-10xx, symbol SW_Push
- removed SW12, SW18: S7, Buttons_Switches_THT:SW_TH_Tactile_Omron_B3F-10xx, symbol SW_Push
- removed SW13: S2, Buttons_Switches_THT:SW_TH_Tactile_Omron_B3F-10xx, symbol SW_Push
- removed SW15, SW16, SW19, SW20, SW23, SW24: SW_Push, Buttons_Switches_THT:SW_TH_Tactile_Omron_B3F-10xx, symbol SW_Push
- removed SW17: S3, Buttons_Switches_THT:SW_TH_Tactile_Omron_B3F-10xx, symbol SW_Push
- removed SW2: Repeat, Buttons_Switches_THT:SW_PUSH-12mm, symbol SW_Push
- removed SW21: S4, Buttons_Switches_THT:SW_TH_Tactile_Omron_B3F-10xx, symbol SW_Push
- removed SW22: S8, Buttons_Switches_THT:SW_TH_Tactile_Omron_B3F-10xx, symbol SW_Push
- removed SW3: Save, Buttons_Switches_THT:SW_TH_Tactile_Omron_B3F-10xx, symbol SW_Push
- removed SW4: Mutate, Buttons_Switches_THT:SW_PUSH-12mm, symbol SW_Push
- removed SW5: Shift, Buttons_Switches_THT:SW_TH_Tactile_Omron_B3F-10xx, symbol SW_Push
- removed SW6: GlideBtn, Buttons_Switches_THT:SW_TH_Tactile_Omron_B3F-10xx, symbol SW_Push
- removed SW7: Play, Buttons_Switches_THT:SW_TH_Tactile_Omron_B3F-10xx, symbol SW_Push
- removed SW9: S1, Buttons_Switches_THT:SW_TH_Tactile_Omron_B3F-10xx, symbol SW_Push
- added C10, C14: 100pF, Capacitors_THT:C_Disc_D3.8mm_W2.6mm_P2.50mm, symbol Device:C
- added C11, C12, C8: 47uF, Capacitors_THT:CP_Radial_D6.3mm_P2.50mm, symbol Device:CP1
- added C13, C15, C16, C9: 100nF, Capacitors_THT:C_Disc_D5.0mm_W2.5mm_P2.50mm, symbol Device:C
- added C18, C19: 47uF, Capacitors_THT:CP_Radial_D6.3mm_P2.50mm, symbol Device:CP1_Small
- added C3: 1uF, Capacitors_THT:CP_Radial_D4.0mm_P2.00mm, symbol Device:CP1
- added D21: 1N4001, Diodes_THT:D_DO-15_P10.16mm_Horizontal, symbol Device:D
- added D22: D, Diodes_THT:D_DO-15_P10.16mm_Horizontal, symbol Device:D
- added J4: Conn_02x05_Odd_Even, Pin_Headers:Pin_Header_Straight_2x05_Pitch2.54mm, symbol Connector_Generic:Conn_02x05_Odd_Even
- added J5: ICSP Header, Pin_Headers:Pin_Header_Straight_2x03_Pitch2.54mm, symbol Connector_Generic:Conn_02x03_Odd_Even
- added J9: BA56_3DIG_7SEG, Eurocad:BA56_3DIG_7SEG, symbol eurocad:BA56_3DIG_7SEG
- added L2, L3: L, Inductors_THT:L_Axial_L5.3mm_D2.2mm_P7.62mm_Horizontal_Vishay_IM-1, symbol Device:L
- added Q1, Q2, Q6, Q7: 2N7000, TO_SOT_Packages_THT:TO-92_Inline_Narrow_Oval, symbol Transistor_FET:2N7000
- added Q8, Q9: 2N3904, TO_SOT_Packages_THT:TO-92_Inline_Narrow_Oval, symbol Transistor_BJT:2N3904
- added R10, R11, R12, R13, R14, R15, R16, R17, R18, R19, R9: 1K, Resistors_THT:R_Axial_DIN0207_L6.3mm_D2.5mm_P7.62mm_Horizontal, symbol Device:R
- added R30, R38: 10k, Resistors_THT:R_Axial_DIN0207_L6.3mm_D2.5mm_P10.16mm_Horizontal, symbol Device:R
- added R36, R42: 1M, Resistors_THT:R_Axial_DIN0207_L6.3mm_D2.5mm_P10.16mm_Horizontal, symbol Device:R
- added R4: 1M, Resistors_THT:R_Axial_DIN0207_L6.3mm_D2.5mm_P7.62mm_Horizontal, symbol Device:R
- added R41: 100k, Resistors_THT:R_Axial_DIN0207_L6.3mm_D2.5mm_P10.16mm_Horizontal, symbol Device:R
- added S1, S10, S11, S12, S13, S14, S15, S16, S2, S3, S4, S5, S6, S7, S8, S9: SW, Buttons_Switches_THT:SW_TH_Tactile_Omron_B3F-10xx, symbol TactSwitch4Pin:SW
- added S17: Load, Buttons_Switches_THT:SW_TH_Tactile_Omron_B3F-10xx, symbol TactSwitch4Pin:SW
- added S18: Save, Buttons_Switches_THT:SW_TH_Tactile_Omron_B3F-10xx, symbol TactSwitch4Pin:SW
- added S19: Play, Buttons_Switches_THT:SW_TH_Tactile_Omron_B3F-10xx, symbol TactSwitch4Pin:SW
- added S20: Shift, Buttons_Switches_THT:SW_TH_Tactile_Omron_B3F-10xx, symbol TactSwitch4Pin:SW
- added S23: GlideBtn, Buttons_Switches_THT:SW_TH_Tactile_Omron_B3F-10xx, symbol TactSwitch4Pin:SW
- added SW2: Repeat, Buttons_Switches_THT:SW_PUSH-12mm, symbol Switch:SW_Push
- added SW3: Mutate, Buttons_Switches_THT:SW_PUSH-12mm, symbol Switch:SW_Push
- added U3: LP2950-3.3_TO92, TO_SOT_Packages_THT:TO-92_Inline_Narrow_Oval, symbol Regulator_Linear:LP2950-3.3_TO92
- C1: value 10uf -> 47uF; footprint Capacitors_THT:CP_Radial_D4.0mm_P2.00mm -> Capacitors_THT:CP_Radial_D6.3mm_P2.50mm; symbol CP1 -> Device:CP1
- C17: renamed from C7; value C -> 22pf; footprint (none) -> Capacitors_THT:C_Disc_D3.0mm_W2.0mm_P2.50mm; symbol C -> Device:C
- C2: renamed from C9; symbol C -> Device:C
- C20: renamed from C8; value C -> 22pf; footprint (none) -> Capacitors_THT:C_Disc_D3.0mm_W2.0mm_P2.50mm; symbol C -> Device:C
- C4: renamed from C2; value C -> 100nF; footprint (none) -> Capacitors_THT:C_Disc_D5.0mm_W2.5mm_P2.50mm; symbol C -> Device:C
- C5: value C -> 100nF; footprint (none) -> Capacitors_THT:C_Disc_D5.0mm_W2.5mm_P2.50mm; symbol C -> Device:C
- C6: renamed from C10; footprint Capacitors_THT:C_Disc_D3.0mm_W2.0mm_P2.50mm -> Capacitors_THT:C_Disc_D3.8mm_W2.6mm_P2.50mm; symbol C -> Device:C
- C7: renamed from C6; value C -> 100nF; footprint (none) -> Capacitors_THT:C_Disc_D5.0mm_W2.5mm_P2.50mm; symbol C -> Device:C
- D1: renamed from D5; symbol LED -> Device:LED
- D10: renamed from D11; symbol LED -> Device:LED
- D11: renamed from D16; symbol LED -> Device:LED
- D12: renamed from D20; symbol LED -> Device:LED
- D13: renamed from D8; symbol LED -> Device:LED
- D14: renamed from D12; symbol LED -> Device:LED
- D15: renamed from D17; symbol LED -> Device:LED
- D16: renamed from D21; symbol LED -> Device:LED
- D18: renamed from D3; footprint (none) -> LEDs:LED_D5.0mm; symbol LED -> Device:LED
- D19: renamed from D4; symbol LED -> Device:LED
- D2: renamed from D9; symbol LED -> Device:LED
- D20: renamed from D24; value D -> BAT85; footprint (none) -> Diodes_THT:D_A-405_P7.62mm_Horizontal; symbol D -> Device:D
- D3: renamed from D14; symbol LED -> Device:LED
- D4: renamed from D18; symbol LED -> Device:LED
- D5: renamed from D6; symbol LED -> Device:LED
- D6: renamed from D10; symbol LED -> Device:LED
- D7: renamed from D15; symbol LED -> Device:LED
- D8: renamed from D19; symbol LED -> Device:LED
- D9: renamed from D7; symbol LED -> Device:LED
- J1: renamed from J4; footprint (none) -> Eurocad:PJ301M-12; symbol Audio-Jack-2_Switch -> conn:Audio-Jack-2_Switch
- J2: renamed from J6; footprint (none) -> Eurocad:PJ301M-12; symbol Audio-Jack-2_Switch -> conn:Audio-Jack-2_Switch
- J3, J7: footprint (none) -> Eurocad:PJ301M-12; symbol Audio-Jack-2_Switch -> conn:Audio-Jack-2_Switch
- J6: renamed from J5; footprint (none) -> Eurocad:PJ301M-12; symbol Audio-Jack-2_Switch -> conn:Audio-Jack-2_Switch
- J8: renamed from J2; value Reset -> Reset In; footprint Socket_Strips:Socket_Strip_Angled_1x17_Pitch2.00mm -> Eurocad:PJ301M-12; symbol Audio-Jack-2_Switch -> conn:Audio-Jack-2_Switch
- L1: renamed from L3; footprint Inductors_THT:L_Axial_L6.6mm_D2.7mm_P10.16mm_Horizontal_Vishay_IM-2 -> Inductors_THT:L_Axial_L5.3mm_D2.2mm_P7.62mm_Horizontal_Vishay_IM-1; symbol L -> Device:L
- Q3: renamed from Q1; footprint TO_SOT_Packages_THT:TO-92_Molded_Narrow -> TO_SOT_Packages_THT:TO-92_Inline_Narrow_Oval; symbol 2N3904 -> transistors:2N3904
- Q4: renamed from Q2; footprint TO_SOT_Packages_THT:TO-92_Molded_Narrow -> TO_SOT_Packages_THT:TO-92_Inline_Narrow_Oval; symbol 2N3904 -> transistors:2N3904
- Q5: renamed from Q3; footprint TO_SOT_Packages_THT:TO-92_Molded_Narrow -> TO_SOT_Packages_THT:TO-92_Inline_Narrow_Oval; symbol 2N3904 -> transistors:2N3904
- R1: renamed from R11; value R -> 100; symbol R -> Device:R
- R2: renamed from R26; value R -> 10k; symbol R -> Device:R
- R20: renamed from R15; value 150 -> 100; symbol R -> Device:R
- R21: renamed from R16; value 150 -> 100; symbol R -> Device:R
- R22: renamed from R17; value 150 -> 100; symbol R -> Device:R
- R23: renamed from R18; value 150 -> 100; symbol R -> Device:R
- R24: renamed from R19; value 150 -> 100; symbol R -> Device:R
- R25: renamed from R20; value 150 -> 100; symbol R -> Device:R
- R26: renamed from R21; value 150 -> 100; symbol R -> Device:R
- R27: renamed from R22; value 150 -> 100; symbol R -> Device:R
- R28: renamed from R8; symbol R -> Device:R
- R29: renamed from R7; value R -> 1k; symbol R -> Device:R
- R3: renamed from R12; value R -> 100; symbol R -> Device:R
- R31: renamed from R3; value R -> 1k; symbol R -> Device:R
- R32: renamed from R1; value R -> 10k; symbol R -> Device:R
- R33: renamed from R4; value R -> 10k; symbol R -> Device:R
- R34: renamed from R24; value R -> 100k; symbol R -> Device:R
- R35: renamed from R27; value R -> 1k; symbol R -> Device:R
- R37: renamed from R5; value R -> 1k; symbol R -> Device:R
- R39: renamed from R2; value R -> 47k; symbol R -> Device:R
- R40: renamed from R6; value R -> 10k; symbol R -> Device:R
- R5: renamed from R13; value R -> 100; symbol R -> Device:R
- R6: renamed from R14; value R -> 100; symbol R -> Device:R
- R7: renamed from R9; symbol R -> Device:R
- R8: renamed from R10; symbol R -> Device:R
- RV1, RV2, RV3, RV4: footprint Potentiometers:Potentiometer_Alps_RK09K_Horizontal -> Eurocad:Alpha9mmPot; symbol POT -> Device:POT
- SW1: renamed from SW8; footprint Buttons_Switches_THT:SW_TH_Tactile_Omron_B3F-10xx -> Rotary_Encoder:RotaryEncoder_Alps_EC12E_Vertical_H20mm; symbol Rotary_Encoder -> Device:Rotary_Encoder
- U1: symbol L7805 -> regul:L7805
- U2: renamed from U5; footprint DIL28 -> Housings_DIP:DIP-28_W7.62mm; symbol ATMEGA328P-PU -> atmel:ATMEGA328P-PU
- U4: renamed from U7; footprint Housings_DIP:DIP-28_W15.24mm_LongPads -> Housings_DIP:DIP-28_W7.62mm; symbol MCP23S17 -> microchip:MCP23S17
- U5: renamed from U2; symbol W25Q80DVSN -> Super-Sixteen-v1-rescue:W25Q80DVSN
- U6: footprint Housings_DIP:DIP-28_W15.24mm_LongPads -> Housings_DIP:DIP-28_W7.62mm; symbol MCP23S17 -> microchip:MCP23S17
- U7: renamed from U4; footprint Housings_DIP:DIP-8_W7.62mm_LongPads -> Housings_DIP:DIP-8_W7.62mm; symbol TL072 -> linear:TL072
- U8: renamed from U3; footprint Housings_DIP:DIP-8_W7.62mm_LongPads -> Housings_DIP:DIP-8_W7.62mm; symbol MCP4822 -> adc-dac:MCP4822
- Y1: value Crystal -> 16mHz; footprint Crystals:Crystal_HC49-4H_Vertical -> Crystals:Crystal_HC18-U_Vertical; symbol Crystal -> Device:Crystal
Connections:
- net labels added: +3V3, B0, B1, B2, B3, B4, B5, B6, B7, C1, C2, C3, C4, C5, C6, C7, C8
- wire segments 438 -> 574
- no-connect marks 9 -> 44
Other:
- note added: "LEVEL SHIFTING"
- moved on the sheet: C1, C17, C2, C20, C6, D1, D10, D11, D12, D13, D14, D15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
