File: kicad-cpu-board-smt/kicad-cpu-board-smt.kicad_pcb (KiCad board)
At the start: 2 copper layers, 78.5 x 69 mm, 56 parts, among them J1 ICSP Header, J2 Conn_01x10_Male, J3 Conn_01x16_Female, J4 Conn_02x05_Odd_Even, Q1 2N7002, Q2 2N7002, Q3 2N7002, Q4 2N7002, U1 AMS1117-5.0, U2 AMS1117-3.3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

Commit message: Fixing CPU footprint on SMT board and updating bom + gerbers
Parts:
- U3: value ATmega328-PU -> ATmega328-AU; footprint Housings_QFP:LQFP-32_7x7mm_Pitch0.8mm -> Housings_QFP:TQFP-32_7x7mm_Pitch0.8mm
- moved U3 0.35 mm to (46.4, 46.0)
Connections:
- U3 pad 1: RESET -> ClockIn
- U3 pad 10: Net-(C8-Pad2) -> DIG2
- U3 pad 11: DIG1 -> DIG3
- U3 pad 12: DIG2 -> CS2
- U3 pad 13: DIG3 -> CS1
- U3 pad 14: CS2 -> CS0
- U3 pad 15: CS1 -> MOSI
- U3 pad 16: CS0 -> MISO
- U3 pad 17: MOSI -> SCK
- U3 pad 18: MISO -> Net-(C5-Pad1)
- U3 pad 19: SCK -> (no net)
- U3 pad 2: Net-(D1-Pad1) -> ResetIn
- U3 pad 20: Net-(C5-Pad1) -> +5V
- U3 pad 21: +5V -> GND
- U3 pad 22: GND -> (no net)
- U3 pad 29: (no net) -> RESET
- U3 pad 3: CS3 -> GND
- U3 pad 30: (no net) -> Net-(D1-Pad1)
- U3 pad 31: (no net) -> CS3
- U3 pad 32: (no net) -> Net-(D2-Pad1)
- U3 pad 4: Net-(D2-Pad1) -> +5V
- U3 pad 5: ClockIn -> GND
- U3 pad 6: ResetIn -> +5V
- U3 pad 7: +5V -> Net-(C7-Pad2)
- U3 pad 8: GND -> Net-(C8-Pad2)
- U3 pad 9: Net-(C7-Pad2) -> DIG1
Routing:
- net Net-(D2-Pad1): track 15.1 -> 8.79 mm
- net CS3: track 41.0 -> 35.5 mm
- net +5V: track 216.5 -> 221.4 mm
- net Net-(C7-Pad2): track 24.8 -> 20.1 mm
- net MISO: track 182.7 -> 186.6 mm
- net MOSI: track 185.5 -> 189.2 mm
- net ClockIn: track 41.2 -> 37.7 mm
- net ResetIn: track 36.0 -> 32.8 mm
- net Net-(D1-Pad1): track 13.8 -> 10.6 mm
- net AD1: track 37.5 -> 40.6 mm
- net CS0: track 56.6 -> 53.8 mm
- net CS1: track 87.9 -> 90.2 mm
- net ENC1: track 59.8 -> 57.8 mm
- net ENC2: track 56.1 -> 54.4 mm
- net CS2: track 33.1 -> 34.7 mm
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
Commit message: Tweaking tracerouting
Parts:
- D1, D2, D3, D4: footprint Diodes_SMD:D_SMA_Handsoldering -> Diodes_SMD:D_SMA-SMB_Universal_Handsoldering
- U3: value ATmega328-AU -> ATmega328P-AU
- moved R4 0.50 mm to (47.5, 57.1)
Routing:
- net Net-(D1-Pad1): track 10.6 -> 9.23 mm
- net Net-(D2-Pad1): track 8.79 -> 9.86 mm
- net AD4: track 30.2 -> 31.1 mm
Other:
- board text added: "SUPER SIXTEEN V1.3 SMT"
- board text removed: "SUPER SIXTEEN V1.1 SMT"
