File: kicad-control-board/kicad-control-board.kicad_pcb (KiCad board)
At the start: 2 copper layers, 100 x 110 mm, 99 parts, among them J1 Conn_01x10_Female, J2 Conn_01x16_Male, J3 BA56-12GWA, J4 Gate Out, J5 Clock Out, J6 Clock In, J7 Pitch Out, J8 CV Out, J9 Reset In, Q1 2N3906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

Commit message: Flipping 2n3906 transistors silkscreen
Parts:
- removed REF***: WEEE-Logo_5.6x8mm_SilkScreen, Symbols:WEEE-Logo_5.6x8mm_SilkScreen
- removed REF***: OSHW-Logo2_7.3x6mm_SilkScreen, Symbols:OSHW-Logo2_7.3x6mm_SilkScreen
- added  : WEEE-Logo_5.6x8mm_SilkScreen, Symbols:WEEE-Logo_5.6x8mm_SilkScreen, F.Cu at (62.1, 23.7)
- added   : OSHW-Logo2_7.3x6mm_SilkScreen, Symbols:OSHW-Logo2_7.3x6mm_SilkScreen, F.Cu at (48.9, 23.1)
- J3: value BA56-12GWA -> BA56_3DIG_7SEG
- R14, R15, R16: value 680R -> 680
- R6: value 100R x7 -> 100
- moved Q1 5.08 mm to (33.0, 16.0), turned to 0 degrees
- moved Q2 5.08 mm to (32.9, 22.8), turned to 0 degrees
- moved Q3 5.08 mm to (32.9, 30.2), turned to 0 degrees
Connections:
- Q1 pad 1: Net-(J3-Pad12) -> +5V
- Q1 pad 3: +5V -> Net-(J3-Pad12)
- Q2 pad 1: Net-(J3-Pad9) -> +5V
- Q2 pad 3: +5V -> Net-(J3-Pad9)
- Q3 pad 1: Net-(J3-Pad8) -> +5V
- Q3 pad 3: +5V -> Net-(J3-Pad8)
Other:
- board text added: "SUPER SIXTEEN v2.3"
- board text removed: "SUPER SIXTEEN v2.2"
